File: v3/PCB/v3.brd (EAGLE design)
At the start: 144.7 x 80 mm, 54 parts, among them IC1 MC74HC595ADG, K1 G5Q-1-HA_DC5, K2 G5Q-1-HA_DC5, K3 G5Q-1-HA_DC5, K4 G5Q-1-HA_DC5, Q1 2N3904TA, Q2 2N3904TA, Q3 2N3904TA, Q4 2N3904TA, Q5 SFH6206-3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

Commit message: v3 PCB routing completed
Parts:
- removed H2: MOUNT-HOLE3.3, holes:3,3
- removed J1, J2: (no value), SparkFun-Connectors:1X04
- C2, C3, C4, C5: value 470nF -> 1uF
- moved H3 164.0 mm to (127.3, 4.88)
- moved H4 157.6 mm to (127.4, 48.0)
- moved H1 106.6 mm to (6.55, 6.40)
- moved IC1 50.5 mm to (123.4, 19.5)
- moved C1 46.5 mm to (40.8, 5.12), turned to 315 degrees
- moved NODEMCU 42.8 mm to (119.8, 27.4), turned to 180 degrees
- moved R3 29.1 mm to (80.0, 11.1), turned to 0 degrees
- moved R20 27.7 mm to (97.1, 8.94), turned to 0 degrees
- moved R15 27.6 mm to (81.6, 14.0)
- moved R2 27.4 mm to (62.3, 12.7), turned to 90 degrees
- moved R6 27.2 mm to (15.4, 17.5), turned to 270 degrees
- moved AC_IN 26.8 mm to (8.38, 49.9)
- moved C4 26.8 mm to (65.8, 12.8)
- moved C5 26.8 mm to (86.1, 15.6)
- moved D1 26.8 mm to (39.1, 18.4)
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Connections:
- removed net GND_1: NODEMCU.10
- removed net GND_3: NODEMCU.17
- removed net S1: J2.4, NODEMCU.29
- removed net S2: J2.3, NODEMCU.28
- removed net S3: J2.2, NODEMCU.23
- removed net S4: J2.1, NODEMCU.22
- net GND: now also NODEMCU.10, NODEMCU.17
- net SNS1: now also NODEMCU.29; no longer J1.1
- net SNS2: now also NODEMCU.28; no longer J1.2
- net SNS3: now also NODEMCU.23; no longer J1.3
- net SNS4: now also NODEMCU.22; no longer J1.4
Routing:
- net VDD: track 23.1 -> 170.8 mm, vias 1 -> 6
- net R1: track 0.00 -> 103.3 mm
- net VCC: track 99.6 -> 197.8 mm, vias 0 -> 1
- net R2: track 0.00 -> 77.0 mm
- net R3: track 0.00 -> 54.9 mm
- net SNS3: track 20.2 -> 53.6 mm, vias 0 -> 2
- net SNS2: track 62.7 -> 94.8 mm
- net R4: track 0.00 -> 31.8 mm
- net SNS1: track 73.5 -> 102.5 mm
- net DATA_IN: track 0.00 -> 26.6 mm
- net LATCH: track 0.00 -> 24.9 mm
- net SNS4: track 12.3 -> 35.9 mm
- net CLK: track 0.00 -> 22.2 mm, vias 0 -> 2
- net LOAD4: track 4.73 -> 24.1 mm
- net NTRL: track 31.0 -> 45.3 mm
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- added copper zone on layer 1, net GND
- added copper zone on layer 16, net GND
Other:
- board size 144.7 x 80 mm -> 134.1 x 53.2 mm
- board text added: "S.M.A.R.T Rev 3.0"

Commit message: OE pulled up
Parts:
- added R16: 10K, SparkFun-Resistors:0603
Connections:
- new net OE: IC1.13, NODEMCU.19, R16.1
- net GND: no longer IC1.13
- net VDD: now also R16.2
Routing:
- net OE: track 0.00 -> 36.0 mm, vias 0 -> 1
- net VDD: track 170.8 -> 174.5 mm, vias 6 -> 7
Changed lines of the file:
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@@
 <drawing>
 <settings>
-<setting alwaysvectorfont="yes"/>
+<setting alwaysvectorfont="no"/>
 <setting verticaltext="up"/>
 </settings>
@@
 <attribute name="VALUE" x="126.2888" y="19.1008" size="1.27" layer="28" rot="MR90" align="center"/>
 </element>
+<element name="R16" library="SparkFun-Resistors" package="0603" value="10K" x="124.3584" y="19.304" smashed="yes" rot="R180">
+<attribute name="NAME" x="124.3584" y="18.542" size="0.6096" layer="25" font="vector" ratio="20" rot="R180" align="bottom-center"/>
+<attribute name="PROD_ID" value="RES-07856" x="124.3584" y="19.304" size="1.778" layer="27" rot="R180" display="off"/>
+<attribute name="VALUE" x="124.3584" y="20.066" size="0.6096" layer="27" font="vector" ratio="20" rot="R180" align="top-center"/>
+</element>
 </elements>
 <signals>
@@
 <contactref element="NODEMCU" pad="14"/>
 <contactref element="IC1" pad="8"/>
-<contactref element="IC1" pad="13"/>
 <polygon width="0.4064" layer="16" isolate="0.4064">
 <vertex x="12.5984" y="23.5712"/>
@@
 <wire x1="114.1984" y1="22.352" x2="116.2304" y2="20.32" width="0.4064" layer="16"/>
 <wire x1="116.2304" y1="20.32" x2="119.888" y2="20.32" width="0.4064" layer="16"/>
-<wire x1="119.888" y1="20.32" x2="120.7008" y2="20.32" width="0.4064" layer="16"/>
+<wire x1="119.888" y1="20.32" x2="120.2944" y2="20.32" width="0.4064" layer="16"/>
+<wire x1="120.2944" y1="20.32" x2="120.7008" y2="20.32" width="0.4064" layer="16"/>
 <wire x1="120.2944" y1="20.7264" x2="119.888" y2="20.32" width="0.4064" layer="16"/>
 <wire x1="21.756" y1="17.8816" x2="21.756" y2="16.4728" width="0.4064" layer="16"/>
@@
 <wire x1="111.76" y1="19.7104" x2="110.744" y2="18.6944" width="0.4064" layer="16"/>
 <wire x1="110.744" y1="18.6944" x2="94.2848" y2="18.6944" width="0.4064" layer="16"/>
+<contactref element="R16" pad="2"/>
+<wire x1="123.5084" y1="19.304" x2="122.7328" y2="19.304" width="0.4064" layer="1"/>
+<wire x1="122.7328" y1="19.304" x2="121.7168" y2="20.32" width="0.4064" layer="1"/>
+<wire x1="121.7168" y1="20.32" x2="120.2944" y2="20.32" width="0.4064" layer="1"/>
+<via x="120.2944" y="20.32" extent="1-16" drill="0.35"/>
 </signal>
 <signal name="QC1">
@@
 <wire x1="116.4336" y1="17.272" x2="108.4072" y2="17.272" width="0.4064" layer="16"/>
 </signal>
+<signal name="OE">
+<contactref element="R16" pad="1"/>
+<contactref element="IC1" pad="13"/>
+<wire x1="125.2084" y1="19.304" x2="125.2084" y2="23.7372" width="0.4064" layer="1"/>
+<wire x1="125.2084" y1="23.7372" x2="124.1552" y2="24.7904" width="0.4064" layer="1"/>
+<via x="124.1552" y="24.7904" extent="1-16" drill="0.35"/>
+<wire x1="124.1552" y1="24.7904" x2="124.1552" y2="22.3084" width="0.4064" layer="16"/>
+<wire x1="124.1552" y1="22.3084" x2="124.079" y2="22.2322" width="0.4064" layer="16"/>
+<contactref element="NODEMCU" pad="19"/>
+<wire x1="122.3264" y1="37.592" x2="124.1552" y2="35.7632" width="0.4064" layer="1"/>
+<wire x1="124.1552" y1="35.7632" x2="124.1552" y2="24.7904" width="0.4064" layer="1"/>
+<wire x1="108.4072" y1="37.592" x2="122.3264" y2="37.592" width="0.4064" layer="1"/>
+</signal>
 </signals>

Commit message: OE connected to D0 pin
Connections:
- net OE: now also NODEMCU.30; no longer NODEMCU.19
Routing:
- net OE: track 36.0 -> 33.1 mm
Changed lines of the file:
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@@
 <wire x1="124.1552" y1="24.7904" x2="124.1552" y2="22.3084" width="0.4064" layer="16"/>
 <wire x1="124.1552" y1="22.3084" x2="124.079" y2="22.2322" width="0.4064" layer="16"/>
-<contactref element="NODEMCU" pad="19"/>
-<wire x1="122.3264" y1="37.592" x2="124.1552" y2="35.7632" width="0.4064" layer="1"/>
-<wire x1="124.1552" y1="35.7632" x2="124.1552" y2="24.7904" width="0.4064" layer="1"/>
-<wire x1="108.4072" y1="37.592" x2="122.3264" y2="37.592" width="0.4064" layer="1"/>
+<contactref element="NODEMCU" pad="30"/>
+<wire x1="108.4072" y1="9.652" x2="122.0216" y2="9.652" width="0.4064" layer="1"/>
+<wire x1="125.2084" y1="12.8388" x2="125.2084" y2="19.304" width="0.4064" layer="1"/>
+<wire x1="122.0216" y1="9.652" x2="125.2084" y2="12.8388" width="0.4064" layer="1"/>
 </signal>
 </signals>

Commit message: PCB OE updated
Parts:
- moved R16 10.5 mm to (119.5, 28.7), flipped to the bottom, turned to 0 degrees
Routing:
- net OE: track 33.1 -> 44.2 mm
- net VDD: track 174.5 -> 183.3 mm
- net N$13: track 0.00 -> 2.49 mm
Changed lines of the file:
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@@
 <drawing>
 <settings>
-<setting alwaysvectorfont="no"/>
+<setting alwaysvectorfont="yes"/>
 <setting verticaltext="up"/>
 </settings>
@@
 <attribute name="VALUE" x="126.2888" y="19.1008" size="1.27" layer="28" rot="MR90" align="center"/>
 </element>
-<element name="R16" library="SparkFun-Resistors" package="0603" value="10K" x="124.3584" y="19.304" smashed="yes" rot="R180">
-<attribute name="NAME" x="124.3584" y="18.542" size="0.6096" layer="25" font="vector" ratio="20" rot="R180" align="bottom-center"/>
-<attribute name="PROD_ID" value="RES-07856" x="124.3584" y="19.304" size="1.778" layer="27" rot="R180" display="off"/>
-<attribute name="VALUE" x="124.3584" y="20.066" size="0.6096" layer="27" font="vector" ratio="20" rot="R180" align="top-center"/>
+<element name="R16" library="SparkFun-Resistors" package="0603" value="10K" x="119.4816" y="28.6512" smashed="yes" rot="MR0">
+<attribute name="NAME" x="119.4816" y="29.4132" size="0.6096" layer="26" font="vector" ratio="20" rot="MR0" align="bottom-center"/>
+<attribute name="PROD_ID" value="RES-07856" x="119.4816" y="28.6512" size="1.778" layer="28" rot="MR0" display="off"/>
+<attribute name="VALUE" x="119.4816" y="27.8892" size="0.6096" layer="28" font="vector" ratio="20" rot="MR0" align="top-center"/>
 </element>
 </elements>
@@
 <wire x1="89.408" y1="13.2436" x2="89.408" y2="13.0048" width="0.4064" layer="16"/>
 <via x="121.3104" y="18.8976" extent="1-16" drill="0.35"/>
-<via x="119.6848" y="29.2608" extent="1-16" drill="0.35"/>
+<via x="116.84" y="30.8864" extent="1-16" drill="0.35"/>
 <contactref element="NODEMCU" pad="10"/>
 <contactref element="NODEMCU" pad="17"/>
@@
 <wire x1="116.2304" y1="20.32" x2="119.888" y2="20.32" width="0.4064" layer="16"/>
 <wire x1="119.888" y1="20.32" x2="120.2944" y2="20.32" width="0.4064" layer="16"/>
-<wire x1="120.2944" y1="20.32" x2="120.7008" y2="20.32" width="0.4064" layer="16"/>
 <wire x1="120.2944" y1="20.7264" x2="119.888" y2="20.32" width="0.4064" layer="16"/>
 <wire x1="21.756" y1="17.8816" x2="21.756" y2="16.4728" width="0.4064" layer="16"/>
@@
 <wire x1="110.744" y1="18.6944" x2="94.2848" y2="18.6944" width="0.4064" layer="16"/>
 <contactref element="R16" pad="2"/>
-<wire x1="123.5084" y1="19.304" x2="122.7328" y2="19.304" width="0.4064" layer="1"/>
-<wire x1="122.7328" y1="19.304" x2="121.7168" y2="20.32" width="0.4064" layer="1"/>
-<wire x1="121.7168" y1="20.32" x2="120.2944" y2="20.32" width="0.4064" layer="1"/>
-<via x="120.2944" y="20.32" extent="1-16" drill="0.35"/>
+<wire x1="116.0272" y1="28.6512" x2="114.6048" y2="27.2288" width="0.4064" layer="16"/>
+<wire x1="118.6316" y1="28.6512" x2="116.0272" y2="28.6512" width="0.4064" layer="16"/>
+<via x="114.6048" y="27.2288" extent="1-16" drill="0.35"/>
+<wire x1="108.4072" y1="22.352" x2="109.728" y2="22.352" width="0.4064" layer="1"/>
+<wire x1="109.728" y1="22.352" x2="114.6048" y2="27.2288" width="0.4064" layer="1"/>
 </signal>
 <signal name="QC1">
@@
 <contactref element="R16" pad="1"/>
 <contactref element="IC1" pad="13"/>
-<wire x1="125.2084" y1="19.304" x2="125.2084" y2="23.7372" width="0.4064" layer="1"/>
-<wire x1="125.2084" y1="23.7372" x2="124.1552" y2="24.7904" width="0.4064" layer="1"/>
-<via x="124.1552" y="24.7904" extent="1-16" drill="0.35"/>
-<wire x1="124.1552" y1="24.7904" x2="124.1552" y2="22.3084" width="0.4064" layer="16"/>
 <wire x1="124.1552" y1="22.3084" x2="124.079" y2="22.2322" width="0.4064" layer="16"/>
 <contactref element="NODEMCU" pad="30"/>
-<wire x1="108.4072" y1="9.652" x2="122.0216" y2="9.652" width="0.4064" layer="1"/>
-<wire x1="125.2084" y1="12.8388" x2="125.2084" y2="19.304" width="0.4064" layer="1"/>
-<wire x1="122.0216" y1="9.652" x2="125.2084" y2="12.8388" width="0.4064" layer="1"/>
+<wire x1="124.079" y1="27.305" x2="124.079" y2="22.2322" width="0.4064" layer="16"/>
+<wire x1="120.3316" y1="28.6512" x2="122.7328" y2="28.6512" width="0.4064" layer="16"/>
+<wire x1="122.7328" y1="28.6512" x2="124.079" y2="27.305" width="0.4064" layer="16"/>
+<via x="123.952" y="28.8544" extent="1-16" drill="0.35"/>
+<wire x1="108.4072" y1="9.652" x2="120.8024" y2="9.652" width="0.4064" layer="1"/>
+<wire x1="120.8024" y1="9.652" x2="124.1552" y2="13.0048" width="0.4064" layer="1"/>
+<wire x1="124.1552" y1="13.0048" x2="124.1552" y2="28.6512" width="0.4064" layer="1"/>
+<wire x1="124.1552" y1="28.6512" x2="123.952" y2="28.8544" width="0.4064" layer="1"/>
+<wire x1="123.952" y1="28.8544" x2="124.079" y2="28.7274" width="0.4064" layer="16"/>
+<wire x1="124.079" y1="28.7274" x2="124.079" y2="27.305" width="0.4064" layer="16"/>
+</signal>
+<signal name="N$13">
+<wire x1="122.936" y1="28.6512" x2="123.952" y2="28.6512" width="0.4064" layer="16"/>
+<wire x1="123.952" y1="28.6512" x2="123.7488" y2="28.448" width="0.4064" layer="16"/>
+<wire x1="123.7488" y1="28.448" x2="123.7488" y2="28.0416" width="0.4064" layer="16"/>
+<wire x1="123.7488" y1="27.8384" x2="123.7488" y2="28.0416" width="0.4064" layer="16"/>
+<wire x1="123.7488" y1="28.0416" x2="123.3424" y2="28.448" width="0.4064" layer="16"/>
 </signal>
 </signals>
